Commit message: [PicMobileWonho] cpp test

File: shopee_ros2/src/pickee_mobile_wonho/urdf/robot_core.xacro (robot description, xacro)
@@ -202,5 +202,5 @@
             <origin xyz="0 0 0" rpy="0 0 0"/>
             <geometry>
-                <mesh filename="package://pickee_mobile/meshes/visual/lidar.dae" scale="1 1 1"/>
+                <mesh filename="package://pickee_mobile_wonho/meshes/visual/lidar.dae" scale="1 1 1"/>
             </geometry>
             <material name="blue"/>
@@ -209,5 +209,5 @@
             <origin xyz="0 0 0" rpy="0 0 0"/>
             <geometry>
-                <mesh filename="package://pickee_mobile/meshes/collision/lidar.stl" scale="1 1 1"/>
+                <mesh filename="package://pickee_mobile_wonho/meshes/collision/lidar.stl" scale="1 1 1"/>
             </geometry>
         </collision>

Commit message: [PicMobileWonho] plaaner changed

File: shopee_ros2/src/pickee_mobile_wonho/urdf/robot_core.xacro (robot description, xacro)
@@ -202,5 +202,5 @@
             <origin xyz="0 0 0" rpy="0 0 0"/>
             <geometry>
-                <mesh filename="package://pickee_mobile_wonho/meshes/visual/lidar.dae" scale="1 1 1"/>
+                <mesh filename="/home/wonho/tech_research/Shopee/shopee_ros2/src/pickee_mobile_wonho/meshes/visual/lidar.dae" scale="1 1 1"/>
             </geometry>
             <material name="blue"/>
@@ -209,5 +209,5 @@
             <origin xyz="0 0 0" rpy="0 0 0"/>
             <geometry>
-                <mesh filename="package://pickee_mobile_wonho/meshes/collision/lidar.stl" scale="1 1 1"/>
+                <mesh filename="/home/wonho/tech_research/Shopee/shopee_ros2/src/pickee_mobile_wonho/meshes/collision/lidar.stl" scale="1 1 1"/>
             </geometry>
         </collision>
