Commit message: [PicMobile] 라이다 180도 회전

File: shopee_ros2/src/pickee_mobile/urdf/robot_core.xacro (robot description, xacro)
@@ -243,5 +243,5 @@
         <parent link="${prefix}lidar_mount"/>
         <child link="${prefix}laser_link"/>
-        <origin xyz="0.0 0 0.03" rpy="0 0 0"/>
+        <origin xyz="0.0 0 0.03" rpy="0 0 ${pi}"/>
     </joint>
 </robot>

Commit message: [PicMobileWonho] lidar sensor check

File: shopee_ros2/src/pickee_mobile/urdf/robot_core.xacro (robot description, xacro)
@@ -243,5 +243,6 @@
         <parent link="${prefix}lidar_mount"/>
         <child link="${prefix}laser_link"/>
-        <origin xyz="0.0 0 0.03" rpy="0 0 ${pi}"/>
+        <origin xyz="0.0 0 0.03" rpy="0 0 ${pi - 0.1203450186}"/>
+        <!-- <origin xyz="0.0 0 0.03" rpy="0 0 ${pi}"/> -->
     </joint>
 </robot>

Commit message: [PickeeMobile] 목적지 도착 이후 회전 보정 추가, 실패

File: shopee_ros2/src/pickee_mobile/urdf/robot_core.xacro (robot description, xacro)
@@ -243,5 +243,5 @@
         <parent link="${prefix}lidar_mount"/>
         <child link="${prefix}laser_link"/>
-        <origin xyz="0.0 0 0.03" rpy="0 0 ${pi - 0.1203450186}"/>
+        <origin xyz="0.0 0 0.03" rpy="0 0 ${pi}"/>
         <!-- <origin xyz="0.0 0 0.03" rpy="0 0 ${pi}"/> -->
     </joint>
